Commit message: feat(session-10): add base_footprint root link and IMU sensor to ugv_pt URDF
- Add base_footprint link + fixed joint (z=0.125 m) as Nav2-required root
- Update diff-drive child_frame_id to robot_001/base_footprint
- Add imu_link/imu_joint + Gazebo IMU sensor at 200 Hz on /robot_001/imu/data
- Wire IMU gz-ros bridge in sim_launch.py
- Update base_frame_id in both nav2_params.yaml copies to robot_001/base_footprint

Co-Authored-By: Claude Sonnet 4.6 <noreply@anthropic.com>

File: src/nav_fleet/urdf/ugv_pt.urdf.xacro (robot description, xacro)
@@ -11,4 +11,11 @@
   <xacro:property name="wheel_x_offset" value="0.10"/>
   <!-- ══ LINKS ══════════════════════════════════════════════════════════ -->
+  <!-- base_footprint: 2-D projection of robot on the floor, required by Nav2 -->
+  <link name="base_footprint"/>
+  <joint name="base_footprint_joint" type="fixed">
+    <parent link="base_footprint"/>
+    <child link="base_link"/>
+    <origin xyz="0 0 0.125" rpy="0 0 0"/>
+  </joint>
   <!-- Base body -->
   <link name="base_link">
@@ -135,4 +142,23 @@
     <origin xyz="${base_length/2} 0 ${base_height/2 + 0.015}"/>
   </joint>
+  <!-- IMU -->
+  <link name="imu_link">
+    <inertial>
+      <mass value="0.01"/>
+      <inertia ixx="0.00001" ixy="0" ixz="0" iyy="0.00001" iyz="0" izz="0.00001"/>
+    </inertial>
+  </link>
+  <joint name="imu_joint" type="fixed">
+    <parent link="base_link"/>
+    <child link="imu_link"/>
+    <origin xyz="0 0 0.05" rpy="0 0 0"/>
+  </joint>
+  <gazebo reference="imu_link">
+    <sensor name="imu" type="imu">
+      <topic>/robot_001/imu/data</topic>
+      <update_rate>200</update_rate>
+      <always_on>true</always_on>
+    </sensor>
+  </gazebo>
   <!-- ══ GAZEBO COLOURS ═════════════════════════════════════════════════
        OGRE2 in Gazebo Harmonic needs <diffuse> for visible surface colour
@@ -195,5 +221,5 @@
       <tf_topic>/robot_001/tf</tf_topic>
       <frame_id>robot_001/odom</frame_id>
-      <child_frame_id>robot_001/base_link</child_frame_id>
+      <child_frame_id>robot_001/base_footprint</child_frame_id>
     </plugin>
     <plugin filename="gz-sim-pose-publisher-system"

Commit message: feat(session-10): first passing nav tests — BR-01, BR-02, BR-10 green
Root cause of multi-session "robot won't turn" bug: the diff-drive plugin
only drove the rear two wheel joints. Passive front wheels resisted in-place
rotation via lateral friction. Odom (computed from driven-wheel joint
positions) falsely reported rotation while the body stayed stationary.

Fix: include all four wheel joints in gz-sim-diff-drive-system.

Other Nav2 changes locked in this session:
- Planner: NavFn → SMAC 2D (equal diagonal cost → true NNE paths)
- RPP: use_collision_detection:false, rotate_to_heading_min_angle:0.3
- Camera visual/collision removed: GPU lidar self-returns caused
  collision_monitor to zero all cmd_vel
- Green sphere goal marker added at (0.0, 3.7) in bedroom_simple.sdf
- Spawn: y=1.5 → y=1.2 (outer hallway arch)
- sim_launch_minimal.py + direct_drive_test.py added as diagnostics

Co-Authored-By: Claude Sonnet 4.6 <noreply@anthropic.com>

File: src/nav_fleet/urdf/ugv_pt.urdf.xacro (robot description, xacro)
@@ -76,5 +76,5 @@
     <axis xyz="0 0 1"/>
   </joint>
-  <!-- Front left wheel (passive — fixed joint, gives 4-wheel UGV appearance) -->
+  <!-- Front left wheel (passive — continuous joint, freewheels under ground contact) -->
   <link name="front_left_wheel">
     <visual>
@@ -90,10 +90,11 @@
     </inertial>
   </link>
-  <joint name="front_left_wheel_joint" type="fixed">
+  <joint name="front_left_wheel_joint" type="continuous">
     <parent link="base_link"/>
     <child link="front_left_wheel"/>
     <origin xyz="${wheel_x_offset} ${wheel_separation/2} -${base_height/2}" rpy="-1.5708 0 0"/>
-  </joint>
-  <!-- Front right wheel (passive — fixed joint) -->
+    <axis xyz="0 0 1"/>
+  </joint>
+  <!-- Front right wheel (passive — continuous joint, freewheels under ground contact) -->
   <link name="front_right_wheel">
     <visual>
@@ -109,8 +110,9 @@
     </inertial>
   </link>
-  <joint name="front_right_wheel_joint" type="fixed">
+  <joint name="front_right_wheel_joint" type="continuous">
     <parent link="base_link"/>
     <child link="front_right_wheel"/>
     <origin xyz="${wheel_x_offset} -${wheel_separation/2} -${base_height/2}" rpy="-1.5708 0 0"/>
+    <axis xyz="0 0 1"/>
   </joint>
   <!-- LiDAR -->
@@ -128,8 +130,8 @@
     <origin xyz="0.05 0 ${base_height/2 + 0.025}"/>
   </joint>
-  <!-- Camera -->
+  <!-- Camera — no visual/collision geometry: GPU lidar uses visual mesh for ray casting,
+       so any geometry here appears as a self-return inside the footprint and causes
+       the collision_monitor to zero all cmd_vel. Camera sensor is in the gazebo block below. -->
   <link name="camera_link">
-    <visual><geometry><box size="0.02 0.08 0.03"/></geometry></visual>
-    <collision><geometry><box size="0.02 0.08 0.03"/></geometry></collision>
     <inertial>
       <mass value="0.1"/>
@@ -202,10 +204,4 @@
     </material>
   </gazebo>
-  <gazebo reference="camera_link">
-    <material>
-      <ambient>0.08 0.08 0.08 1</ambient>
-      <diffuse>0.12 0.12 0.12 1</diffuse>
-    </material>
-  </gazebo>
   <!-- ══ GAZEBO PLUGINS ══════════════════════════════════════════════════ -->
   <gazebo>
@@ -213,5 +209,7 @@
             name="gz::sim::systems::DiffDrive">
       <left_joint>rear_left_wheel_joint</left_joint>
+      <left_joint>front_left_wheel_joint</left_joint>
       <right_joint>rear_right_wheel_joint</right_joint>
+      <right_joint>front_right_wheel_joint</right_joint>
       <wheel_separation>${wheel_separation}</wheel_separation>
       <wheel_radius>${wheel_radius}</wheel_radius>

Commit message: fix: ugv_pt.urdf.xacro footprint — 350x300mm -> real 253x231mm
RealRobotStartup.md A2's footprint-verification checklist item. Read the vendor
drawing (docs/img/waveshare_ugv_pt_dimensions.png) directly rather than trust the
doc's prior transcription -- confirmed 253x231mm footprint, 289mm height w/ mast,
126mm wheelbase, 25.13mm ground clearance are all accurate.

base_length/base_width were 0.35/0.30 (350x300mm), a real ~38%/~30% oversize
with no basis found anywhere -- corrected to 0.253/0.231. Sim-collision-geometry
only: Nav2's real-robot safety footprint (nav2_params.yaml robot_radius=0.24, a
480mm circle) is separate and independently confirmed still adequate (real
chassis half-diagonal ~0.171m < 0.24m, ~69mm margin) -- no change needed there.

wheel_separation/wheel_x_offset deliberately NOT touched -- the 6-wheel-skid-
steer-vs-4-wheel-diff-drive kinematic mismatch is a separate, already-known/
accepted gap (EKF is its mitigation), out of scope for this footprint-only fix.

Verified xacro still processes the file cleanly (exit 0) and emits the corrected
box size; full local suite (534 tests) still green. Not pushed.

Co-Authored-By: Claude Sonnet 5 <noreply@anthropic.com>

File: src/nav_fleet/urdf/ugv_pt.urdf.xacro (robot description, xacro)
@@ -2,6 +2,17 @@
 <robot name="ugv_pt" xmlns:xacro="http://www.ros.org/wiki/xacro">
   <xacro:property name="base_mass" value="5.0"/>
-  <xacro:property name="base_length" value="0.35"/>
-  <xacro:property name="base_width" value="0.30"/>
+  <!-- 0.253/0.231 (253x231mm) — corrected 2026-08-10 against the real vendor drawing
+       (docs/img/waveshare_ugv_pt_dimensions.png, read directly, not from memory) —
+       was 0.35/0.30 (350x300mm), a real ~38%/~30% oversize with no basis found
+       anywhere. Sim-collision-geometry-only: Nav2's own real-robot safety footprint
+       (nav2_params.yaml robot_radius=0.24) is separate and was independently
+       confirmed still adequate (real chassis half-diagonal ~0.171m < 0.24m) —
+       this fix is about sim/real visual + collision-physics parity, not navigation
+       safety. wheel_separation/wheel_x_offset below are NOT touched here — the
+       6-wheel-skid-steer-vs-4-wheel-diff-drive kinematic mismatch is a separate,
+       already-known/accepted gap (EKF is its mitigation), out of scope for this
+       footprint-only fix. -->
+  <xacro:property name="base_length" value="0.253"/>
+  <xacro:property name="base_width" value="0.231"/>
   <xacro:property name="base_height" value="0.15"/>
   <xacro:property name="wheel_radius" value="0.05"/>
